File: Schematic/V2/V2.kicad_sch (KiCad schematic)
At the start: 11 parts, among them J1 OUT1, J2 OUT2, J3 OUT3, J4 OUT4, J5 OUT5, U1 ESP32-S2

Commit message: Added V2
Parts:
- removed U1: ESP32-S2, Package_DFN_QFN:QFN-56-1EP_7x7mm_P0.4mm_EP4x4mm, symbol MCU_Espressif:ESP32-S2
- added J6: 5V ESP, Connector_Wire:SolderWire-0.25sqmm_1x02_P4.2mm_D0.65mm_OD1.7mm_Relief, symbol Connector_Generic:Conn_01x02
- added J7: 5V LEDS, Connector_Wire:SolderWire-0.25sqmm_1x02_P4.2mm_D0.65mm_OD1.7mm_Relief, symbol Connector_Generic:Conn_01x02
- added U1: ~, WEMOS-ESP32-S2:WEMOS-ESP32-S2, symbol WEMOS-ESP32-S2:WEMOS-ESP32-S2
- F1, F2, F3, F4, F5: footprint (none) -> KiCad:1812L010DR
- J1, J2, J3, J4, J5: footprint (none) -> Connector_Wire:SolderWire-0.25sqmm_1x03_P4.2mm_D0.65mm_OD1.7mm_Relief
Connections:
- net GND: now also J6.2 (Pin_2), J7.2 (Pin_2), U1.23 (GND), U1.31 (GND)
- net OUT1: now also U1.9 (GPIO1)
- net OUT2: now also U1.10 (GPIO2)
- net OUT3: now also U1.2 (GPIO3)
- net OUT4: now also U1.11 (GPIO4)
- net OUT5: now also U1.30 (GPIO16)
- net OUT5V1: now reaches F1.2, J1.1 (Pin_1)
- net OUT5V2: now reaches F2.2, J2.1 (Pin_1)
- net OUT5V5: now reaches F5.2, J5.1 (Pin_1)
- net OUT5V4: now reaches F4.2, J4.1 (Pin_1)
- net OUT5V3: now reaches F3.2, J3.1 (Pin_1)
- net +5V renamed +5V2
- net +5V2: now also J7.1 (Pin_1)
- new net +5V1: J6.1 (Pin_1), U1.32 (VBUS)
Other:
- moved on the sheet: F1, F2, F3, F4, F5, J1, J2, J3, J4, J5

Commit message: Added support for two 18 AWG wires as 5V input to allow 14A and updated traces as needed.
Parts:
- removed J7: 5V LEDS, Connector_Wire:SolderWire-0.25sqmm_1x02_P4.2mm_D0.65mm_OD1.7mm_Relief, symbol Connector_Generic:Conn_01x02
- added J7: 5V LEDS, Connector_Wire:SolderWire-0.75sqmm_1x04_P4.8mm_D1.25mm_OD2.3mm_Relief, symbol Connector_Generic:Conn_01x04
Connections:
- net +5V2: now also J7.1 (Pin_1), J7.2 (Pin_2)
- net GND: now also J7.3 (Pin_3), J7.4 (Pin_4)
Changed lines of the file:
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@@
+	(symbol
+		(lib_id "power:+5V")
+		(at 87.63 81.28 90)
+		(unit 1)
+		(exclude_from_sim no)
+		(in_bom yes)
+		(on_board yes)
+		(dnp no)
+		(fields_autoplaced yes)
+		(property "Reference" "#PWR018"
+			(at 91.44 81.28 0)
+			(effects
+				(font
+					(size 1.27 1.27)
+				)
+				(hide yes)
+			)
+		)
+		(property "Value" "+5V2"
+			(at 83.82 81.2799 90)
+			(effects
+				(font
+					(size 1.27 1.27)
+				)
+				(justify left)
+			)
+		)
+		(property "Footprint" ""
+			(at 87.63 81.28 0)
+			(effects
+				(font
+					(size 1.27 1.27)
+				)
+				(hide yes)
+			)
+		)
+		(property "Datasheet" ""
+			(at 87.63 81.28 0)
+			(effects
+				(font
+					(size 1.27 1.27)
+				)
+				(hide yes)
+			)
+		)
+		(property "Description" "Power symbol creates a global label with name \"+5V\""
+			(at 87.63 81.28 0)
+			(effects
+				(font
+					(size 1.27 1.27)
+				)
+				(hide yes)
+			)
+		)
+		(pin "1"
+		)
+		(instances
+			(project "V2"
+				(path "/7c1fabcd-e970-4249-87b0-60c290ed6e5c"
+					(reference "#PWR018")
+					(unit 1)
+				)
+			)
+		)
+	)
 	(symbol
 		(lib_id "power:+5V")
@@
 	)
 	(symbol
+		(lib_id "power:GND")
+		(at 87.63 86.36 270)
+		(unit 1)
+		(exclude_from_sim no)
+		(in_bom yes)
+		(on_board yes)
+		(dnp no)
+		(fields_autoplaced yes)
+		(property "Reference" "#PWR019"
+			(at 81.28 86.36 0)
+			(effects
+				(font
+					(size 1.27 1.27)
+				)
+				(hide yes)
+			)
+		)
+		(property "Value" "GND"
+			(at 83.82 86.3599 90)
+			(effects
+				(font
+					(size 1.27 1.27)
+				)
+				(justify right)
+			)
+		)
+		(property "Footprint" ""
+			(at 87.63 86.36 0)
+			(effects
+				(font
+					(size 1.27 1.27)
+				)
+				(hide yes)
+			)
+		)
+		(property "Datasheet" ""
+			(at 87.63 86.36 0)
+			(effects
+				(font
+					(size 1.27 1.27)
+				)
+				(hide yes)
+			)
+		)
+		(property "Description" "Power symbol creates a global label with name \"GND\" , ground"
+			(at 87.63 86.36 0)
+			(effects
+				(font
+					(size 1.27 1.27)
+				)
+				(hide yes)
+			)
+		)
+		(pin "1"
+		)
+		(instances
+			(project "V2"
+				(path "/7c1fabcd-e970-4249-87b0-60c290ed6e5c"
+					(reference "#PWR019")
+					(unit 1)
+				)
+			)
+		)
+	)
+	(symbol
 		(lib_id "Device:Polyfuse_Small")
 		(at 85.09 40.64 90)
@@
 	)
 	(symbol
+		(lib_id "Connector_Generic:Conn_01x04")
+		(at 92.71 81.28 0)
+		(unit 1)
+		(exclude_from_sim no)
+		(in_bom yes)
+		(on_board yes)
+		(dnp no)
+		(fields_autoplaced yes)
+		(property "Reference" "J7"
+			(at 95.25 81.2799 0)
+			(effects
+				(font
+					(size 1.27 1.27)
+				)
+				(justify left)
+			)
+		)
+		(property "Value" "5V LEDS"
+			(at 95.25 83.8199 0)
+			(effects
+				(font
+					(size 1.27 1.27)
+				)
+				(justify left)
+			)
+		)
+		(property "Footprint" "Connector_Wire:SolderWire-0.75sqmm_1x04_P4.8mm_D1.25mm_OD2.3mm_Relief"
+			(at 92.71 81.28 0)
+			(effects
+				(font
+					(size 1.27 1.27)
+				)
+				(hide yes)
+			)
+		)
+		(property "Datasheet" "~"
+			(at 92.71 81.28 0)
+			(effects
+				(font
+					(size 1.27 1.27)
+				)
+				(hide yes)
+			)
+		)
+		(property "Description" "Generic connector, single row, 01x04, script generated (kicad-library-utils/schlib/autogen/connector/)"
+			(at 92.71 81.28 0)
+			(effects
+				(font
+					(size 1.27 1.27)
+				)
+				(hide yes)
+			)
+		)
+		(pin "3"
+		)
+		(pin "1"
+		)
+		(pin "4"
+		)
+		(pin "2"
+		)
+		(instances
+			(project ""
+				(path "/7c1fabcd-e970-4249-87b0-60c290ed6e5c"
+					(reference "J7")
+					(unit 1)
+				)
+			)
+		)
+	)
+	(symbol
 		(lib_id "power:GND")
 		(at 82.55 25.4 270)
@@
 	(symbol
 		(lib_id "power:GND")
-		(at 87.63 81.28 270)
+		(at 87.63 83.82 270)
 		(unit 1)
 		(exclude_from_sim no)
@@
 		(fields_autoplaced yes)
 		(property "Reference" "#PWR014"
-			(at 81.28 81.28 0)
+			(at 81.28 83.82 0)
 			(effects
 				(font
@@
 		)
 		(property "Value" "GND"
-			(at 83.82 81.2799 90)
+			(at 83.82 83.8199 90)
 			(effects
 				(font
@@
 		)
 		(property "Footprint" ""
-			(at 87.63 81.28 0)
+			(at 87.63 83.82 0)
 			(effects
 				(font
@@
 		)
 		(property "Datasheet" ""
-			(at 87.63 81.28 0)
+			(at 87.63 83.82 0)
 			(effects
 				(font
@@
 		)
 		(property "Description" "Power symbol creates a global label with name \"GND\" , ground"
-			(at 87.63 81.28 0)
+			(at 87.63 83.82 0)
 			(effects
 				(font
@@
 					(unit 1)
 				)
-			)
-		)
-	)
-	(symbol
-		(lib_id "Connector_Generic:Conn_01x02")
-		(at 92.71 78.74 0)
-		(unit 1)
-		(exclude_from_sim no)
-		(in_bom yes)
-		(on_board yes)
-		(dnp no)
-		(fields_autoplaced yes)
-		(property "Reference" "J7"
-			(at 95.25 78.7399 0)
-			(effects
-				(font
-					(size 1.27 1.27)
-				)
-				(justify left)
-			)
-		)
-		(property "Value" "5V LEDS"
-			(at 95.25 81.2799 0)
-			(effects
-				(font
-					(size 1.27 1.27)
-				)
-				(justify left)
-			)
-		)
-		(property "Footprint" "Connector_Wire:SolderWire-0.25sqmm_1x02_P4.2mm_D0.65mm_OD1.7mm_Relief"
-			(at 92.71 78.74 0)
-			(effects
-				(font
-					(size 1.27 1.27)
-				)
-				(hide yes)
-			)
-		)
-		(property "Datasheet" "~"
-			(at 92.71 78.74 0)
-			(effects
-				(font
-					(size 1.27 1.27)
-				)
-				(hide yes)
-			)
-		)
-		(property "Description" "Generic connector, single row, 01x02, script generated (kicad-library-utils/schlib/autogen/connector/)"
-			(at 92.71 78.74 0)
-			(effects
-				(font
-					(size 1.27 1.27)
-				)
-				(hide yes)
-			)
-		)
-		(pin "2"
-		)
-		(pin "1"
-		)
-		(instances
-			(project "V2"
-				(path "/7c1fabcd-e970-4249-87b0-60c290ed6e5c"
-					(reference "J7")
-					(unit 1)
-				)
